File: AlienWhoopF7.sch (EAGLE design)
At the start: 51 parts, among them IC1 STM32F4/F7, M1 53047-0210, M2 53047-0210, M3 53047-0210, M4 53047-0210, Q1 IRLML6402, Q2 FDMA410NZ, Q3 FDMA410NZ, Q4 FDMA410NZ, Q5 FDMA410NZ, U1 TPS63001, U2 MPU-9250, Y1 8mhz

Commit message: Updated to V2.1 with Blackbox
Parts:
- removed CAM: VTX, AlienWhoop:TINYPADS
- removed LS1: RCX03-787, AlienWhoop:RCX03-787
- removed MYLED1, MYLED2, MYLED3, MYLED4: CUSTOM, alienflight:SMD-CHIP-LED-0805
- removed RX: SBUS, alienflight:JST-ZR_3-PIN
- removed SJ1: BOOT, AlienWhoop:TINYPADS
- removed SJ2: BIND, AlienWhoop:TINYPADS
- removed UART4: RXTX, AlienWhoop:TINYPADS
- removed VBAT: VBAT, AlienWhoop:TINYPADS
- added 3.3V, 3V3, BOOT, GND, GND@1, RX2, RX2/INV, RX3, RX4, TX2, TX3, TX4, VCC@1: TESTPAD, AlienWhoop:TESTPAD
- added U3: MX25L6406EM2I-12G, AlienWhoop:M25P32
- added U4: SN74LVC1G04DBVR, AlienWhoop:SN74LVC1G04
- BAT: BOM (none) -> EXCLUDE
- IC1: value STM32F4/F7 -> STM32F405RGT
- L1: device alienflight:NR301X -> AlienWhoop:DFE201612E-2R2M-P2; PARTNO (none) -> DFE201612E-2R2M-P2
- LOGO3: BOM (none) -> EXCLUDE; PARTNO (none) -> OSHW-LOGOS
- Q2, Q3, Q4, Q5: value FDMA410NZ -> FDMA410NZT; PARTNO (none) -> FDMA410NZT
- U2: value MPU-9250 -> MPU-6500; PARTNO (none) -> MPU-6500
- USB: value 105133-0011-SD -> 614105150621; device AlienWhoop:MICROUSB1051330011-SD-VIAS -> AlienWhoop:MICROUSBUSB-BFPV; PARTNO (none) -> 614105150621
- renumbered PWR to POWER
Connections:
- removed net BIND: IC1MCU.PC13, SJ2.1
- removed net F4F7_INCOMPAT_26: IC1MCU.PB0
- removed net F4F7_INCOMPAT_27: IC1MCU.PB1
- removed net F4F7_INCOMPAT_28: IC1MCU.PB2
- removed net F4F7_INCOMPAT_29: IC1MCU.PB10
- removed net I2C1_SCL: IC1MCU.PB6
- removed net I2C1_SDA: IC1MCU.PB7
- removed net SPI2_MISO: IC1MCU.PB14
- removed net SPI2_MOSI: IC1MCU.PB15
- removed net SPI2_NSS: IC1MCU.PB12
- removed net SPI2_SCK: IC1MCU.PB13
- new net INV_SBUS: RX2/INV.1, U4.A
- net 3.3V: now also 3.3V.1, 3V3.1, U3.RST, U3.VCC, U3.WP, U4.VCC; no longer MYLED1.A, MYLED2.A, MYLED3.A, MYLED4.A, RX.1, SJ1.1
- net BOOT0: now also BOOT.1; no longer SJ1.2
- net GND: now also GND.1, GND@1.1, IC1MCU.PA13, IC1MCU.PA14, IC1MCU.PA8, IC1MCU.PB0, IC1MCU.PB1, IC1MCU.PB10, IC1MCU.PB12, IC1MCU.PB13, IC1MCU.PB14, IC1MCU.PB15, IC1MCU.PB2, IC1MCU.PB6, IC1MCU.PB7, IC1MCU.PB8, IC1MCU.PB9, IC1MCU.PC0, IC1MCU.PC1, IC1MCU.PC13, IC1MCU.PC15, IC1MCU.PC2, IC1MCU.PC3, IC1MCU.PC4, U3.VSS, U4.GND; no longer CAM.2, LS1.2, MYLED1.C, MYLED2.C, MYLED3.C, MYLED4.C, RX.2, SJ2.2, VBAT.2
- net SPI3_MISO: now also U3.OUT
- net SPI3_MOSI: now also U3.IN
- net SPI3_NSS: now also IC1MCU.PA15, U3.CS; no longer IC1MCU.PC15
- net SPI3_SCK: now also U3.CLK
- net UART2_RX: now also RX2.1, U4.Y
- net UART2_TX: now also TX2.1; no longer LS1.1
- net UART3_RX: now also RX3.1; no longer RX.3
- net UART3_TX: now also TX3.1
- net UART4_RX: now also RX4.1; no longer UART4.1
- net UART4_TX: now also TX4.1; no longer UART4.2
- net VCC: now also VCC@1.1; no longer CAM.1, VBAT.1
Other:
- note added: "Battery Connector"
- note added: "EX BIND"
- note added: "F4 BOOT1"
- note added: "Jumper"
- note added: "Motor Outputs"
- note added: "Remixed from AlienFlight F3 Brushed Quad http://alienflight.com/f3-brushed-quad/"
- note added: "Sbux Rx, Dataflash (Blackbox)"
- note added: "THIRD DRAFT"
- note added: "http://www.alienwhoop.us/git/"
- note added: "https://www.facebook.com/alienwhoop/"
- note added: "v20180608A"
- note removed: "*NOT JUMPER"
- note removed: "Beeper, Camera/VTX, and Sbus Rx"
- note removed: "Brushed Motor Power (9.5A Continuous 24A Pulsed FETs)"
- note removed: "CUSTOM LED 3.3V PADS"
- note removed: "DIY MIX"
- note removed: "PowerWhoop Pigtail"
- note removed: "Remixed from AlienFlight F3 Brushed Quad http://f3-quad.alienwhoop.us/"
- note removed: "http://fb.me/alienwhoop/"
- note removed: "http://git.alienwhoop.us/"
- note removed: "v20170807A"
- moved on the sheet: C2, C3, C5, U2
